Commit message: Fix wrong frame of STL files

File: ass1/urdf/manmaru.urdf.xacro (robot description, xacro)
@@ -1,7 +1,7 @@
 <?xml version="1.0"?>
 <robot name="manmaru" xmlns:xacro="http://ros.org/wiki/xacro">
-  <xacro:macro name="wheel_inertial" params="mass">
+  <xacro:macro name="default_inertial" params="mass">
     <inertial>
-      <origin xyz="0.05 0 -0.03" rpy="0 0 0"/>
+      <origin xyz="0 0 0" rpy="0 0 0"/>
       <mass value="${mass}" />
       <inertia ixx="1.0" ixy="0.0" ixz="0.0" iyy="1.0" iyz="0.0" izz="1.0" />
@@ -22,11 +22,11 @@
         </geometry>
       </collision>
-      <xacro:wheel_inertial mass="1"/>
+      <xacro:default_inertial mass="1"/>
     </link>
     <joint name="${prefix}_wheel_joint" type="continuous">
+      <origin xyz="${x} ${y} 0" rpy="0 0 0"/>
       <axis xyz="0 1 0" rpy="0 0 0" />
       <parent link="trunk"/>
       <child link="${prefix}_wheel"/>
-      <origin xyz="${x} ${y} 0" rpy="0 0 0"/>
     </joint>
     <!-- This block provides Gazebo with information on a few additional physical properties. -->
@@ -52,5 +52,5 @@
   <link name="trunk">
     <visual>
-      <origin xyz="0.05 0 0" rpy="${pi/2} 0 0" />
+      <origin xyz="0 0 0" rpy="0 0 0" />
       <geometry>
         <mesh filename="package://ass1/meshes/trunk.stl"/>
@@ -58,14 +58,10 @@
     </visual>
     <collision>
-      <origin xyz="0.05 0 0" rpy="${pi/2} 0 0" />
+      <origin xyz="0 0 0" rpy="0 0 0" />
       <geometry>
         <mesh filename="package://ass1/meshes/trunk.stl"/>
       </geometry>
     </collision>
-    <inertial>
-      <origin xyz="0.05 0 -0.02" rpy="${pi/2} 0 0"/>
-      <mass value="5" />
-      <inertia ixx="1.0" ixy="0.0" ixz="0.0" iyy="1.0" iyz="0.0" izz="1.0" />
-    </inertial>
+    <xacro:default_inertial mass="5"/>
   </link>
   <joint name="dummy_joint" type="fixed">
@@ -73,8 +69,8 @@
     <child link="trunk"/>
   </joint>
-  <xacro:wheel prefix="left_front"  x="0.05"  y="0.06"/>
-  <xacro:wheel prefix="left_back"   x="0.05"  y="-0.06"/>
-  <xacro:wheel prefix="right_front" x="-0.05" y="0.06"/>
-  <xacro:wheel prefix="right_back"  x="-0.05" y="-0.06"/>
+  <xacro:wheel prefix="left_front"  x="0.04"  y="0.04"/>
+  <xacro:wheel prefix="left_back"   x="0.04"  y="-0.04"/>
+  <xacro:wheel prefix="right_front" x="-0.04" y="0.04"/>
+  <xacro:wheel prefix="right_back"  x="-0.04" y="-0.04"/>
   <!-- Gazebo plugin for ROS Control -->
   <gazebo>

Commit message: Place LiDAR on trunk of manmaru

File: ass1/urdf/manmaru.urdf.xacro (robot description, xacro)
@@ -49,4 +49,5 @@
     </transmission>
   </xacro:macro>
+  <!-- Trunk -->
   <link name="dummy"></link>
   <link name="trunk">
@@ -69,8 +70,30 @@
     <child link="trunk"/>
   </joint>
+  <!-- Four Wheels -->
   <xacro:wheel prefix="left_front"  x="0.04"  y="0.04"/>
   <xacro:wheel prefix="left_back"   x="0.04"  y="-0.04"/>
   <xacro:wheel prefix="right_front" x="-0.04" y="0.04"/>
   <xacro:wheel prefix="right_back"  x="-0.04" y="-0.04"/>
+  <!-- LiDAR -->
+  <link name="rplidar">
+    <visual>
+      <origin xyz="0 0 0" rpy="${pi/2} 0 ${pi}" />
+      <geometry>
+        <mesh filename="package://ass1/meshes/rplidar.stl" scale="0.0002 0.0002 0.0002"/>
+      </geometry>
+    </visual>
+    <collision>
+      <origin xyz="0 0 0" rpy="${pi/2} 0 ${pi}" />
+      <geometry>
+        <mesh filename="package://ass1/meshes/rplidar.stl" scale="0.0002 0.0002 0.0002"/>
+      </geometry>
+    </collision>
+    <xacro:default_inertial mass="0.1"/>
+  </link>
+  <joint name="rplidar" type="fixed">
+    <origin xyz="0.04 -0.007 0.015" rpy="0 0 0"/>
+    <parent link="trunk"/>
+    <child link="rplidar"/>
+  </joint>
   <!-- Gazebo plugin for ROS Control -->
   <gazebo>

Commit message: Add mobile manipulator

File: ass1/urdf/manmaru.urdf.xacro (robot description, xacro)
@@ -76,9 +76,9 @@
   <xacro:wheel prefix="right_back"  x="-0.04" y="-0.04"/>
   <!-- LiDAR -->
-  <link name="rplidar">
+  <link name="lidar">
     <visual>
       <origin xyz="0 0 0" rpy="${pi/2} 0 ${pi}" />
       <geometry>
-        <mesh filename="package://ass1/meshes/rplidar.stl" scale="0.0002 0.0002 0.0002"/>
+        <mesh filename="package://ass1/meshes/lidar.stl" scale="0.0002 0.0002 0.0002"/>
       </geometry>
     </visual>
@@ -86,14 +86,274 @@
       <origin xyz="0 0 0" rpy="${pi/2} 0 ${pi}" />
       <geometry>
-        <mesh filename="package://ass1/meshes/rplidar.stl" scale="0.0002 0.0002 0.0002"/>
+        <mesh filename="package://ass1/meshes/lidar.stl" scale="0.0002 0.0002 0.0002"/>
       </geometry>
     </collision>
     <xacro:default_inertial mass="0.1"/>
   </link>
-  <joint name="rplidar" type="fixed">
+  <joint name="lidar_on_trunk" type="fixed">
     <origin xyz="0.04 -0.007 0.015" rpy="0 0 0"/>
     <parent link="trunk"/>
-    <child link="rplidar"/>
-  </joint>
+    <child link="lidar"/>
+  </joint>
+  <!-- Mobile Manipulator -->
+  <xacro:arg name="lamp" default="false"/>
+  <xacro:arg name="gripper" default="true"/>
+  <link name="long_U">
+    <visual>
+      <origin xyz="0 0 0" rpy="0 0 0" />
+      <geometry>
+        <mesh filename="package://ass1/meshes/mobile_manipulator/long_U.dae" scale="0.7 0.7 0.7"/>
+      </geometry>
+    </visual>
+    <collision>
+      <origin xyz="0 0 0" rpy="0 0 0" />
+      <geometry>
+        <mesh filename="package://ass1/meshes/mobile_manipulator/long_U.dae" scale="0.7 0.7 0.7"/>
+      </geometry>
+    </collision>
+    <inertial>
+      <mass value="0.1" />
+      <inertia ixx="0.03" iyy="0.03" izz="0.03" ixy="0.0" ixz="0.0" iyz="0.0" />
+    </inertial>
+  </link>
+  <joint name="m1" type="continuous">
+    <origin xyz="-0.02 0 0.015" rpy="0 0 ${pi/2}" />
+    <parent link="trunk" />
+    <child link="long_U" />
+    <axis xyz="0 0 1" />
+  </joint>
+  <link name="section_1">
+    <visual>
+      <origin xyz="0 0 0" rpy="0 1.5707963267949 0" />
+      <geometry>
+        <mesh filename="package://ass1/meshes/mobile_manipulator/section_1.dae" scale="0.7 0.7 0.7"/>
+      </geometry>
+    </visual>
+    <collision>
+      <origin xyz="0 0 0" rpy="0 1.5707963267949 0" />
+      <geometry>
+        <mesh filename="package://ass1/meshes/mobile_manipulator/section_1.dae" scale="0.7 0.7 0.7"/>
+      </geometry>
+    </collision>
+    <inertial>
+      <mass value="0.1" />
+      <inertia ixx="0.03" iyy="0.03" izz="0.03" ixy="0.0" ixz="0.0" iyz="0.0" />
+    </inertial>
+  </link>
+  <joint name="m2" type="continuous">
+    <origin xyz="0 0 0.017" rpy="0 -1.5707963267949 0" />
+    <parent link="long_U" />
+    <child link="section_1" />
+    <axis xyz="0 0 -1" />
+  </joint>
+  <link name="section_2">
+    <visual>
+      <origin xyz="0 0 0" rpy="0 1.5707963267949 0" />
+      <geometry>
+        <mesh filename="package://ass1/meshes/mobile_manipulator/section_2.dae" scale="0.7 0.7 0.7"/>
+      </geometry>
+    </visual>
+    <collision>
+      <origin xyz="0 0 0" rpy="0 1.5707963267949 0" />
+      <geometry>
+        <mesh filename="package://ass1/meshes/mobile_manipulator/section_2.dae" scale="0.7 0.7 0.7"/>
+      </geometry>
+    </collision>
+    <inertial>
+      <mass value="0.1" />
+      <inertia ixx="0.03" iyy="0.03" izz="0.03" ixy="0.0" ixz="0.0" iyz="0.0" />
+    </inertial>
+  </link>
+  <joint name="m3" type="continuous">
+    <origin xyz="0.038 0 0" rpy="0 0 0" />
+    <parent link="section_1" />
+    <child link="section_2" />
+    <axis xyz="0 0 -1" />
+  </joint>
+  <link name="section_3">
+    <visual>
+      <origin xyz="0 0 0" rpy="0 3.14159268 0" />
+      <geometry>
+        <mesh filename="package://ass1/meshes/mobile_manipulator/section_3.dae" scale="0.7 0.7 0.7"/>
+      </geometry>
+    </visual>
+    <collision>
+      <origin xyz="0 0 0" rpy="0 3.14159268 0" />
+      <geometry>
+        <mesh filename="package://ass1/meshes/mobile_manipulator/section_3.dae" scale="0.7 0.7 0.7"/>
+      </geometry>
+    </collision>
+    <inertial>
+      <mass value="0.1" />
+      <inertia ixx="0.03" iyy="0.03" izz="0.03" ixy="0.0" ixz="0.0" iyz="0.0" />
+    </inertial>
+  </link>
+  <joint name="m4" type="continuous">
+    <origin xyz="0.031 0 0" rpy="0 -1.5707963267949 0" />
+    <parent link="section_2" />
+    <child link="section_3" />
+    <axis xyz="0 0 -1" />
+  </joint>
+  <link name="section_4">
+    <visual>
+      <xacro:if value="$(arg lamp)">
+        <origin xyz="0 0 0" rpy="0 -1.5707963267949 1.5707963267949" />
+        <geometry>
+          <mesh filename="package://ass1/meshes/mobile_manipulator/section_1.dae" scale="0.7 0.7 0.7"/>
+        </geometry>
+      </xacro:if>
+      <xacro:if value="$(arg gripper)">
+        <origin xyz="0 -0.058 0" rpy="0 -1.5707963267949 0" />
+        <geometry>
+          <mesh filename="package://ass1/meshes/mobile_manipulator/section_4.dae" scale="0.7 0.7 0.7"/>
+        </geometry>
+      </xacro:if>
+    </visual>
+    <collision>
+      <origin xyz="0 -0.035 0" rpy="1.5707963267949 0 0" />
+      <geometry>
+        <cylinder length="0.06" radius="0.02" />
+        <box size="0.05 0.02 0.03" />
+      </geometry>
+    </collision>
+    <inertial>
+      <mass value="0.1" />
+      <inertia ixx="0.03" iyy="0.03" izz="0.03" ixy="0.0" ixz="0.0" iyz="0.0" />
+    </inertial>
+  </link>
+  <joint name="m5" type="continuous">
+    <origin xyz="0 -0.033 0" rpy="0 -1.5707963267949 0" />
+    <parent link="section_3" />
+    <child link="section_4" />
+    <axis xyz="0 0 1" />
+  </joint>
+  <link name="fixed_tip" />
+  <joint name="t7f" type="fixed">
+    <xacro:if value="$(arg lamp)">
+      <origin xyz="0 -0.075 0" rpy="-1.5707963267949 0 0" />
+      <parent link="section_5" />
+    </xacro:if>
+    <xacro:if value="$(arg gripper)">
+      <origin xyz="0 -0.11 0" rpy="-1.5707963267949 0 0" />
+      <parent link="section_4" />
+    </xacro:if>
+    <child link="fixed_tip" />
+  </joint>
+  <link name="section_5">
+    <xacro:if value="$(arg lamp)">
+      <visual>
+        <origin xyz="0 0 0" rpy="0 0 1.5707963267949" />
+        <geometry>
+          <mesh filename="package://ass1/meshes/mobile_manipulator/lamp.dae" scale="0.7 0.7 0.7"/>
+        </geometry>
+      </visual>
+      <collision>
+        <origin xyz="0 -0.045 0" rpy="1.5707963267949 0 0" />
+        <geometry>
+          <cylinder length="0.06" radius="0.03" />
+          <box size="0.05 0.02 0.03" />
+        </geometry>
+      </collision>
+    </xacro:if>
+    <xacro:if value="$(arg gripper)">
+      <visual>
+        <origin xyz="0 0 0" rpy="0 0 0" />
+        <geometry>
+          <mesh filename="package://ass1/meshes/mobile_manipulator/gripper.dae" scale="0.7 0.7 0.7"/>
+        </geometry>
+      </visual>
+      <collision>
+        <origin xyz="0 0 0" rpy="0 0 0" />
+        <geometry>
+          <mesh filename="package://ass1/meshes/mobile_manipulator/gripper.dae" scale="0.7 0.7 0.7"/>
+        </geometry>
+      </collision>
+    </xacro:if>
+    <inertial>
+      <mass value="0.1" />
+      <inertia ixx="0.03" iyy="0.03" izz="0.03" ixy="0.0" ixz="0.0" iyz="0.0" />
+    </inertial>
+  </link>
+  <joint name="m6" type="continuous">
+    <xacro:if value="$(arg lamp)">
+      <origin xyz="0 -0.054 0" rpy="0 0 0" />
+      <axis xyz="0 0 1" />
+    </xacro:if>
+    <xacro:if value="$(arg gripper)">
+      <origin xyz="0 -0.058 0" rpy="0 -1.5707963267949 0" />
+      <axis xyz="0 0 -1" />
+    </xacro:if>
+    <parent link="section_4" />
+    <child link="section_5" />
+  </joint>
+  <xacro:if value="$(arg gripper)">
+    <link name="moving_tip" />
+    <joint name="t7m" type="fixed">
+      <origin xyz="0 -0.052 0" rpy="-1.5707963267949 0 0" />
+      <parent link="section_5" />
+      <child link="moving_tip" />
+    </joint>
+  </xacro:if>
+  <transmission name="trans_m1">
+    <type>transmission_interface/SimpleTransmission</type>
+    <joint name="m1">
+      <!-- TODO: Why EffortJointInterface yeids fluctuation? -->
+      <hardwareInterface>hardware_interface/VelocityJointInterface</hardwareInterface>
+    </joint>
+    <actuator name="m1_motor">
+      <hardwareInterface>hardware_interface/VelocityJointInterface</hardwareInterface>
+      <mechanicalReduction>1</mechanicalReduction>
+    </actuator>
+  </transmission>
+  <transmission name="trans_m2">
+    <type>transmission_interface/SimpleTransmission</type>
+    <joint name="m2">
+      <hardwareInterface>hardware_interface/VelocityJointInterface</hardwareInterface>
+    </joint>
+    <actuator name="m2_motor">
+      <hardwareInterface>hardware_interface/VelocityJointInterface</hardwareInterface>
+      <mechanicalReduction>1</mechanicalReduction>
+    </actuator>
+  </transmission>
+  <transmission name="trans_m3">
+    <type>transmission_interface/SimpleTransmission</type>
+    <joint name="m3">
+      <hardwareInterface>hardware_interface/VelocityJointInterface</hardwareInterface>
+    </joint>
+    <actuator name="m3_motor">
+      <hardwareInterface>hardware_interface/VelocityJointInterface</hardwareInterface>
+      <mechanicalReduction>1</mechanicalReduction>
+    </actuator>
+  </transmission>
+  <transmission name="trans_m4">
+    <type>transmission_interface/SimpleTransmission</type>
+    <joint name="m4">
+      <hardwareInterface>hardware_interface/VelocityJointInterface</hardwareInterface>
+    </joint>
+    <actuator name="m4_motor">
+      <hardwareInterface>hardware_interface/VelocityJointInterface</hardwareInterface>
+      <mechanicalReduction>1</mechanicalReduction>
+    </actuator>
+  </transmission>
+  <transmission name="trans_m5">
+    <type>transmission_interface/SimpleTransmission</type>
+    <joint name="m5">
+      <hardwareInterface>hardware_interface/VelocityJointInterface</hardwareInterface>
+    </joint>
+    <actuator name="m5_motor">
+      <hardwareInterface>hardware_interface/VelocityJointInterface</hardwareInterface>
+      <mechanicalReduction>1</mechanicalReduction>
+    </actuator>
+  </transmission>
+  <transmission name="trans_m6">
+    <type>transmission_interface/SimpleTransmission</type>
+    <joint name="m6">
+      <hardwareInterface>hardware_interface/VelocityJointInterface</hardwareInterface>
+    </joint>
+    <actuator name="m6_motor">
+      <hardwareInterface>hardware_interface/VelocityJointInterface</hardwareInterface>
+      <mechanicalReduction>1</mechanicalReduction>
+    </actuator>
+  </transmission>
   <!-- Gazebo plugin for ROS Control -->
   <gazebo>
