Commit message: Navi half completed

File: manmaru_description/urdf/lidar.urdf.xacro (robot description, xacro)
@@ -14,9 +14,8 @@
          </geometry>
       </collision>
-      <xacro:default_inertial mass="0.1"/>
    </link>
-   <joint name="lidar_on_trunk" type="fixed">
+   <joint name="lidar_on_base" type="fixed">
       <origin xyz="0.04 -0.007 0.015" rpy="0 0 0"/>
-      <parent link="trunk"/>
+      <parent link="classis"/>
       <child link="lidar_link"/>
    </joint>

File: manmaru_description/urdf/manipulator.urdf.xacro (robot description, xacro)
@@ -23,5 +23,5 @@
    <joint name="m1" type="continuous">
       <origin xyz="-0.02 0 0.015" rpy="0 0 ${pi/2}" />
-      <parent link="trunk" />
+      <parent link="classis" />
       <child link="long_U" />
       <axis xyz="0 0 1" />

File: manmaru_description/urdf/manmaru.urdf.xacro (robot description, xacro)
@@ -1,11 +1,4 @@
 <?xml version="1.0"?>
 <robot name="manmaru" xmlns:xacro="http://ros.org/wiki/xacro">
-   <xacro:macro name="default_inertial" params="mass">
-      <inertial>
-         <origin xyz="0 0 0" rpy="0 0 0"/>
-         <mass value="${mass}" />
-         <inertia ixx="1.0" ixy="0.0" ixz="0.0" iyy="1.0" iyz="0.0" izz="1.0" />
-      </inertial>
-   </xacro:macro>
    <xacro:macro name="wheel" params="prefix x y">
       <link name="${prefix}_wheel">
@@ -22,38 +15,38 @@
             </geometry>
          </collision>
-         <xacro:default_inertial mass="1"/>
+         <!-- Mass and inertia matrix are generated by Onshape's mass properties tool -->
+         <!-- Material: Polyurethane -->
+         <inertial>
+            <origin
+               xyz="0 0 0"
+               rpy="0 0 0" />
+            <mass
+               value="0.022" />
+            <inertia
+               ixx="3.533e-6"
+               ixy="0"
+               ixz="0"
+               iyy="6.714e-6"
+               iyz="0"
+               izz="3.533e-6" />
+         </inertial>
       </link>
       <joint name="${prefix}_wheel_joint" type="continuous">
          <origin xyz="${x} ${y} 0" rpy="0 0 0"/>
          <axis xyz="0 1 0" rpy="0 0 0" />
-         <parent link="trunk"/>
+         <parent link="classis"/>
          <child link="${prefix}_wheel"/>
       </joint>
-      <!-- This block provides Gazebo with information on a few additional physical properties. -->
-      <gazebo reference="${prefix}_wheel">
-         <mu1 value="200.0"/>
-         <mu2 value="100.0"/>
-         <kp value="1000000.0" />
-         <kd value="10.0" />
-      </gazebo>
-      <!-- This block connects the wheel joint to an actuator (motor), which informs both
-      simulation and visualization of the robot -->
-      <transmission name="${prefix}_wheel_trans">
-         <type>transmission_interface/SimpleTransmission</type>
-         <actuator name="${prefix}_wheel_motor">
-            <mechanicalReduction>1</mechanicalReduction>
-         </actuator>
-         <joint name="${prefix}_wheel_joint">
-            <hardwareInterface>hardware_interface/VelocityJointInterface</hardwareInterface>
-         </joint>
-      </transmission>
    </xacro:macro>
-   <!-- Trunk -->
-   <link name="dummy"></link>
-   <link name="trunk">
+   <link name="base_link" />
+   <joint name="base_link_to_chassis" type="fixed">
+      <parent link="base_link"/>
+      <child link="classis"/>
+   </joint>
+   <link name="classis">
       <visual>
          <origin xyz="0 0 0" rpy="0 0 0" />
          <geometry>
-            <mesh filename="package://manmaru_description/meshes/trunk.stl"/>
+            <mesh filename="package://manmaru_description/meshes/base.stl"/>
          </geometry>
       </visual>
@@ -61,18 +54,29 @@
          <origin xyz="0 0 0" rpy="0 0 0" />
          <geometry>
-            <mesh filename="package://manmaru_description/meshes/trunk.stl"/>
+            <mesh filename="package://manmaru_description/meshes/base.stl"/>
          </geometry>
       </collision>
-      <xacro:default_inertial mass="5"/>
+      <!-- Mass and inertia matrix are generated by Onshape's mass properties tool -->
+      <!-- Material: Aluminum -->
+      <inertial>
+         <origin
+            xyz="0 0 0"
+            rpy="0 0 0" />
+         <mass
+            value="0.354" />
+         <inertia
+            ixx="9.785e-5"
+            ixy="-2.359e-10"
+            ixz="0"
+            iyy="2.357e-4"
+            iyz="1.475e-10"
+            izz="2.855e-4" />
+      </inertial>
    </link>
-   <joint name="dummy_joint" type="fixed">
-      <parent link="dummy"/>
-      <child link="trunk"/>
-   </joint>
-   <!-- Four Wheels -->
+   <!-- Four wheels -->
    <xacro:wheel prefix="left_front"  x="0.04"  y="0.04"/>
-   <xacro:wheel prefix="left_back"   x="0.04"  y="-0.04"/>
-   <xacro:wheel prefix="right_front" x="-0.04" y="0.04"/>
-   <xacro:wheel prefix="right_back"  x="-0.04" y="-0.04"/>
+   <xacro:wheel prefix="left_rear"   x="-0.04" y="0.04"/>
+   <xacro:wheel prefix="right_front" x="0.04"  y="-0.04"/>
+   <xacro:wheel prefix="right_rear"  x="-0.04" y="-0.04"/>
    <!-- LiDAR -->
    <xacro:include filename="lidar.urdf.xacro" />

Commit message: Robot does not move as expected
Robot moves too slowly, and its wheels often slip and skid.

Learning about vehicle dynamics might help.

File: manmaru_description/urdf/lidar.urdf.xacro (robot description, xacro)
@@ -5,5 +5,5 @@
          <origin xyz="0 0 0" rpy="${pi/2} 0 ${pi}" />
          <geometry>
-            <mesh filename="package://manmaru_description/meshes/lidar.stl" scale="0.0002 0.0002 0.0002"/>
+            <mesh filename="package://manmaru_description/meshes/lidar.stl" scale="0.002 0.002 0.002"/>
          </geometry>
       </visual>
@@ -11,10 +11,10 @@
          <origin xyz="0 0 0" rpy="${pi/2} 0 ${pi}" />
          <geometry>
-            <mesh filename="package://manmaru_description/meshes/lidar.stl" scale="0.0002 0.0002 0.0002"/>
+            <mesh filename="package://manmaru_description/meshes/lidar.stl" scale="0.002 0.002 0.002"/>
          </geometry>
       </collision>
    </link>
    <joint name="lidar_on_base" type="fixed">
-      <origin xyz="0.04 -0.007 0.015" rpy="0 0 0"/>
+      <origin xyz="0.4 -0.075 0.15" rpy="0 0 0"/>
       <parent link="classis"/>
       <child link="lidar_link"/>

File: manmaru_description/urdf/manipulator.urdf.xacro (robot description, xacro)
@@ -7,5 +7,5 @@
          <origin xyz="0 0 0" rpy="0 0 0" />
          <geometry>
-            <mesh filename="package://manmaru_description/meshes/manipulator/long_U.dae" scale="0.7 0.7 0.7"/>
+            <mesh filename="package://manmaru_description/meshes/manipulator/long_U.dae" scale="5.4 5.4 5.4"/>
          </geometry>
       </visual>
@@ -13,5 +13,5 @@
          <origin xyz="0 0 0" rpy="0 0 0" />
          <geometry>
-            <mesh filename="package://manmaru_description/meshes/manipulator/long_U.dae" scale="0.7 0.7 0.7"/>
+            <mesh filename="package://manmaru_description/meshes/manipulator/long_U.dae" scale="5.4 5.4 5.4"/>
          </geometry>
       </collision>
@@ -22,5 +22,5 @@
    </link>
    <joint name="m1" type="continuous">
-      <origin xyz="-0.02 0 0.015" rpy="0 0 ${pi/2}" />
+      <origin xyz="-0.2 0 0.15" rpy="0 0 ${pi/2}" />
       <parent link="classis" />
       <child link="long_U" />
@@ -31,11 +31,11 @@
          <origin xyz="0 0 0" rpy="0 1.5707963267949 0" />
          <geometry>
-            <mesh filename="package://manmaru_description/meshes/manipulator/section_1.dae" scale="0.7 0.7 0.7"/>
-         </geometry>
-      </visual>
-      <collision>
-         <origin xyz="0 0 0" rpy="0 1.5707963267949 0" />
-         <geometry>
-            <mesh filename="package://manmaru_description/meshes/manipulator/section_1.dae" scale="0.7 0.7 0.7"/>
+            <mesh filename="package://manmaru_description/meshes/manipulator/section_1.dae" scale="5.4 5.4 5.4"/>
+         </geometry>
+      </visual>
+      <collision>
+         <origin xyz="0 0 0" rpy="0 1.5707963267949 0" />
+         <geometry>
+            <mesh filename="package://manmaru_description/meshes/manipulator/section_1.dae" scale="5.4 5.4 5.4"/>
          </geometry>
       </collision>
@@ -46,5 +46,5 @@
    </link>
    <joint name="m2" type="continuous">
-      <origin xyz="0 0 0.017" rpy="0 -1.5707963267949 0" />
+      <origin xyz="0 0 0.13" rpy="0 -1.5707963267949 0" />
       <parent link="long_U" />
       <child link="section_1" />
@@ -55,11 +55,11 @@
          <origin xyz="0 0 0" rpy="0 1.5707963267949 0" />
          <geometry>
-            <mesh filename="package://manmaru_description/meshes/manipulator/section_2.dae" scale="0.7 0.7 0.7"/>
-         </geometry>
-      </visual>
-      <collision>
-         <origin xyz="0 0 0" rpy="0 1.5707963267949 0" />
-         <geometry>
-            <mesh filename="package://manmaru_description/meshes/manipulator/section_2.dae" scale="0.7 0.7 0.7"/>
+            <mesh filename="package://manmaru_description/meshes/manipulator/section_2.dae" scale="5.4 5.4 5.4"/>
+         </geometry>
+      </visual>
+      <collision>
+         <origin xyz="0 0 0" rpy="0 1.5707963267949 0" />
+         <geometry>
+            <mesh filename="package://manmaru_description/meshes/manipulator/section_2.dae" scale="5.4 5.4 5.4"/>
          </geometry>
       </collision>
@@ -70,5 +70,5 @@
    </link>
    <joint name="m3" type="continuous">
-      <origin xyz="0.038 0 0" rpy="0 0 0" />
+      <origin xyz="0.29 0 0" rpy="0 0 0" />
       <parent link="section_1" />
       <child link="section_2" />
@@ -79,5 +79,5 @@
          <origin xyz="0 0 0" rpy="0 3.14159268 0" />
          <geometry>
-            <mesh filename="package://manmaru_description/meshes/manipulator/section_3.dae" scale="0.7 0.7 0.7"/>
+            <mesh filename="package://manmaru_description/meshes/manipulator/section_3.dae" scale="5.4 5.4 5.4"/>
          </geometry>
       </visual>
@@ -85,5 +85,5 @@
          <origin xyz="0 0 0" rpy="0 3.14159268 0" />
          <geometry>
-            <mesh filename="package://manmaru_description/meshes/manipulator/section_3.dae" scale="0.7 0.7 0.7"/>
+            <mesh filename="package://manmaru_description/meshes/manipulator/section_3.dae" scale="5.4 5.4 5.4"/>
          </geometry>
       </collision>
@@ -94,5 +94,5 @@
    </link>
    <joint name="m4" type="continuous">
-      <origin xyz="0.031 0 0" rpy="0 -1.5707963267949 0" />
+      <origin xyz="0.24 0 0" rpy="0 -1.5707963267949 0" />
       <parent link="section_2" />
       <child link="section_3" />
@@ -104,5 +104,5 @@
             <origin xyz="0 0 0" rpy="0 -1.5707963267949 1.5707963267949" />
             <geometry>
-               <mesh filename="package://manmaru_description/meshes/manipulator/section_1.dae" scale="0.7 0.7 0.7"/>
+               <mesh filename="package://manmaru_description/meshes/manipulator/section_1.dae" scale="5.4 5.4 5.4"/>
             </geometry>
          </xacro:if>
@@ -110,5 +110,5 @@
             <origin xyz="0 -0.058 0" rpy="0 -1.5707963267949 0" />
             <geometry>
-               <mesh filename="package://manmaru_description/meshes/manipulator/section_4.dae" scale="0.7 0.7 0.7"/>
+               <mesh filename="package://manmaru_description/meshes/manipulator/section_4.dae" scale="5.4 5.4 5.4"/>
             </geometry>
          </xacro:if>
@@ -127,5 +127,5 @@
    </link>
    <joint name="m5" type="continuous">
-      <origin xyz="0 -0.033 0" rpy="0 -1.5707963267949 0" />
+      <origin xyz="0 -0.51 0" rpy="0 -1.5707963267949 0" />
       <parent link="section_3" />
       <child link="section_4" />
@@ -149,5 +149,5 @@
             <origin xyz="0 0 0" rpy="0 0 1.5707963267949" />
             <geometry>
-               <mesh filename="package://manmaru_description/meshes/manipulator/lamp.dae" scale="0.7 0.7 0.7"/>
+               <mesh filename="package://manmaru_description/meshes/manipulator/lamp.dae" scale="5.4 5.4 5.4"/>
             </geometry>
          </visual>
@@ -164,5 +164,5 @@
             <origin xyz="0 0 0" rpy="0 0 0" />
             <geometry>
-               <mesh filename="package://manmaru_description/meshes/manipulator/gripper.dae" scale="0.7 0.7 0.7"/>
+               <mesh filename="package://manmaru_description/meshes/manipulator/gripper.dae" scale="5.4 5.4 5.4"/>
             </geometry>
          </visual>
@@ -170,5 +170,5 @@
             <origin xyz="0 0 0" rpy="0 0 0" />
             <geometry>
-               <mesh filename="package://manmaru_description/meshes/manipulator/gripper.dae" scale="0.7 0.7 0.7"/>
+               <mesh filename="package://manmaru_description/meshes/manipulator/gripper.dae" scale="5.4 5.4 5.4"/>
             </geometry>
          </collision>
@@ -194,5 +194,5 @@
       <link name="moving_tip" />
       <joint name="t7m" type="fixed">
-         <origin xyz="0 -0.052 0" rpy="-1.5707963267949 0 0" />
+         <origin xyz="0 -0.52 0" rpy="-1.5707963267949 0 0" />
          <parent link="section_5" />
          <child link="moving_tip" />

File: manmaru_description/urdf/manmaru.urdf.xacro (robot description, xacro)
@@ -6,5 +6,5 @@
             <origin xyz="0 0 0" rpy="0 0 0" />
             <geometry>
-               <mesh filename="package://manmaru_description/meshes/wheel.stl"/>
+               <mesh filename="package://manmaru_description/meshes/wheel.stl" />
             </geometry>
          </visual>
@@ -12,5 +12,5 @@
             <origin xyz="0 0 0" rpy="0 0 0" />
             <geometry>
-               <mesh filename="package://manmaru_description/meshes/wheel.stl"/>
+               <mesh filename="package://manmaru_description/meshes/wheel.stl" />
             </geometry>
          </collision>
@@ -22,20 +22,26 @@
                rpy="0 0 0" />
             <mass
-               value="0.022" />
+               value="2.903" />
             <inertia
-               ixx="3.533e-6"
+               ixx="0.058"
                ixy="0"
                ixz="0"
-               iyy="6.714e-6"
+               iyy="0.106"
                iyz="0"
-               izz="3.533e-6" />
+               izz="0.058" />
          </inertial>
       </link>
       <joint name="${prefix}_wheel_joint" type="continuous">
-         <origin xyz="${x} ${y} 0" rpy="0 0 0"/>
+         <origin xyz="${x} ${y} -0.12" rpy="0 0 0"/>
          <axis xyz="0 1 0" rpy="0 0 0" />
          <parent link="classis"/>
          <child link="${prefix}_wheel"/>
       </joint>
+      <!-- <gazebo reference="${prefix}_wheel">
+         <mu1 value="200.0"/>
+         <mu2 value="100.0"/>
+         <kp value="1000000.0" />
+         <kd value="10.0" />
+      </gazebo> -->
    </xacro:macro>
    <link name="base_link" />
@@ -48,5 +54,5 @@
          <origin xyz="0 0 0" rpy="0 0 0" />
          <geometry>
-            <mesh filename="package://manmaru_description/meshes/base.stl"/>
+            <mesh filename="package://manmaru_description/meshes/classis.stl" />
          </geometry>
       </visual>
@@ -54,5 +60,5 @@
          <origin xyz="0 0 0" rpy="0 0 0" />
          <geometry>
-            <mesh filename="package://manmaru_description/meshes/base.stl"/>
+            <mesh filename="package://manmaru_description/meshes/classis.stl" />
          </geometry>
       </collision>
@@ -64,19 +70,19 @@
             rpy="0 0 0" />
          <mass
-            value="0.354" />
+            value="15.816" />
          <inertia
-            ixx="9.785e-5"
-            ixy="-2.359e-10"
-            ixz="0"
-            iyy="2.357e-4"
-            iyz="1.475e-10"
-            izz="2.855e-4" />
+            ixx="0.719"
+            ixy="-4.801e-5"
+            ixz="3.711e-16"
+            iyy="1.456"
+            iyz="5.022e-5"
+            izz="1.735" />
       </inertial>
    </link>
    <!-- Four wheels -->
-   <xacro:wheel prefix="left_front"  x="0.04"  y="0.04"/>
-   <xacro:wheel prefix="left_rear"   x="-0.04" y="0.04"/>
-   <xacro:wheel prefix="right_front" x="0.04"  y="-0.04"/>
-   <xacro:wheel prefix="right_rear"  x="-0.04" y="-0.04"/>
+   <xacro:wheel prefix="left_front"  x="0.4"  y="0.4"/>
+   <xacro:wheel prefix="left_rear"   x="-0.4" y="0.4"/>
+   <xacro:wheel prefix="right_front" x="0.4"  y="-0.4"/>
+   <xacro:wheel prefix="right_rear"  x="-0.4" y="-0.4"/>
    <!-- LiDAR -->
    <xacro:include filename="lidar.urdf.xacro" />
